Commit message: change12

File: src/house/urdf/mybot.gazebo.xacro (robot description, xacro)
@@ -28,6 +28,6 @@
   </gazebo>
   <gazebo reference="ball_wheel_link">
-    <mu1>0.1</mu1>
-    <mu2>0.1</mu2>
+    <mu1>0.4</mu1>
+    <mu2>0.4</mu2>
     <kp>500000.0</kp>
     <kd>100.0</kd>
@@ -60,6 +60,6 @@
       <wheelSeparation>0.180</wheelSeparation>
       <wheelDiameter>0.05</wheelDiameter>
-      <wheelAcceleration>10</wheelAcceleration>
-      <wheelTorque>100</wheelTorque>
+      <wheelAcceleration>1.0</wheelAcceleration>
+      <wheelTorque>5.0</wheelTorque>
       <rosDebugLevel>na</rosDebugLevel>
     </plugin>

File: src/house/urdf/mybot.urdf (robot description, URDF)
Before this commit: robot mybot, 5 links, 4 joints
Links:
- link base_link: mass 0.1 -> 1.0
Joints:
- joint ball_wheel_joint: type fixed -> continuous
- joint left_wheel_joint: axis 0 0 -1 -> 0 1 0
- joint right_wheel_joint: axis 0 0 -1 -> 0 1 0

File: src/house/urdf/mybot.xacro (robot description, xacro)
@@ -11,6 +11,6 @@
     <inertial>
      <origin xyz="0 0 0" rpy="0 0 0"/>
-     <mass value="0.1"/>
-     <inertia ixx="0.0001"  ixy="0"  ixz="0" iyy="0.0001" iyz="0" izz="0.001" />
+     <mass value="1.0"/>
+     <inertia ixx="0.002"  ixy="0"  ixz="0" iyy="0.003" iyz="0" izz="0.005" />
     </inertial>
     <visual>
@@ -52,5 +52,5 @@
   </link>
   <joint name="right_wheel_joint" type="continuous">
-    <axis xyz="0 0 -1"/>
+    <axis xyz="0 1 0"/>
     <parent link="base_link"/>
     <child link="right_wheel_link"/>
@@ -79,5 +79,5 @@
   </link>
   <joint name="left_wheel_joint" type="continuous">
-    <axis xyz="0 0 -1"/>
+    <axis xyz="0 1 0"/>
     <parent link="base_link"/>
     <child link="left_wheel_link"/>
@@ -88,5 +88,5 @@
      <origin xyz="0 0 0" rpy="0 0 0"/>
      <mass value="0.1"/>
-     <inertia ixx="0"  ixy="0"  ixz="0" iyy="0" iyz="0" izz="0" />
+     <inertia ixx="0.0001"  ixy="0"  ixz="0" iyy="0.0001" iyz="0" izz="0.0001" />
     </inertial>
     <visual>
@@ -105,5 +105,5 @@
     </collision>
   </link>
-  <joint name="ball_wheel_joint" type="fixed">
+  <joint name="ball_wheel_joint" type="continuous">
     <axis xyz="0 0 1"/>
     <parent link="base_link"/>

Commit message: change13

File: src/house/urdf/mybot.gazebo.xacro (robot description, xacro)
@@ -8,6 +8,6 @@
   </gazebo>
   <gazebo reference="left_wheel_link">
-    <mu1>0.5</mu1>
-    <mu2>0.5</mu2>
+    <mu1>0.3</mu1>
+    <mu2>0.3</mu2>
     <kp>500000.0</kp>
     <kd>10.0</kd>
@@ -18,6 +18,6 @@
   </gazebo>
   <gazebo reference="right_wheel_link">
-    <mu1>0.5</mu1>
-    <mu2>0.5</mu2>
+    <mu1>0.3</mu1>
+    <mu2>0.3</mu2>
     <kp>500000.0</kp>
     <kd>10.0</kd>
@@ -28,6 +28,6 @@
   </gazebo>
   <gazebo reference="ball_wheel_link">
-    <mu1>0.4</mu1>
-    <mu2>0.4</mu2>
+    <mu1>0.1</mu1>
+    <mu2>0.1</mu2>
     <kp>500000.0</kp>
     <kd>100.0</kd>
@@ -60,6 +60,6 @@
       <wheelSeparation>0.180</wheelSeparation>
       <wheelDiameter>0.05</wheelDiameter>
-      <wheelAcceleration>1.0</wheelAcceleration>
-      <wheelTorque>5.0</wheelTorque>
+      <wheelAcceleration>7.0</wheelAcceleration>
+      <wheelTorque>75.0</wheelTorque>
       <rosDebugLevel>na</rosDebugLevel>
     </plugin>

File: src/house/urdf/mybot.xacro (robot description, xacro)
@@ -52,5 +52,5 @@
   </link>
   <joint name="right_wheel_joint" type="continuous">
-    <axis xyz="0 1 0"/>
+    <axis xyz="0 0 -1"/>
     <parent link="base_link"/>
     <child link="right_wheel_link"/>
@@ -79,5 +79,5 @@
   </link>
   <joint name="left_wheel_joint" type="continuous">
-    <axis xyz="0 1 0"/>
+    <axis xyz="0 0 -1"/>
     <parent link="base_link"/>
     <child link="left_wheel_link"/>
@@ -106,5 +106,5 @@
   </link>
   <joint name="ball_wheel_joint" type="continuous">
-    <axis xyz="0 0 1"/>
+    <axis xyz="0 1 -1"/>
     <parent link="base_link"/>
     <child link="ball_wheel_link"/>

Commit message: change14

File: src/house/urdf/mybot.gazebo.xacro (robot description, xacro)
@@ -109,5 +109,5 @@
         </scan>
         <range>
-          <min>0.120</min>
+          <min>0.125</min>
           <max>12.0</max>
           <resolution>0.015</resolution>

File: src/house/urdf/mybot.urdf (robot description, URDF)
Before this commit: robot mybot, 5 links, 4 joints
Links:
- link base_link: geometry collision box size=0.25 0.16 0.05; visual box size=0.25 0.18 0.05

File: src/house/urdf/mybot.xacro (robot description, xacro)
@@ -16,5 +16,5 @@
     <visual>
       <geometry>
-        <box size="0.25 0.16 0.05"/>
+        <box size="0.25 0.18 0.05"/>
       </geometry>
       <origin rpy="0 0 0" xyz="0 0 0"/>
